Commit message: Add files via upload

File: esercizio6/urdf/robot_kuka.xacro (robot description, xacro)
@@ -1,5 +1,19 @@
 <?xml version="1.0"?>
 <robot name="robot_kuka" xmlns:xacro="http://wiki.ros.org/xacro">
-    <xacro:include filename="$(find esercizio5)/urdf/robot_kuka_macro.xacro" />
+    <xacro:include filename="$(find esercizio6)/urdf/robot_kuka_macro.xacro" />
+<xacro:base_link_macro
+			base_link_name="base_link">
+		</xacro:base_link_macro>
+<xacro:kuka_joint
+			name="joint0"
+			type="prismatic"
+			parent="base_link"
+			child="link1">
+			<origin xyz="0 0 0"/>
+			<axis xyz="1 0 0"/>
+			<orient rpy="0 0 0"/>
+	    <limit effort="176" velocity="0.1" lower="-5" upper="5">
+		</limit>
+		</xacro:kuka_joint>
 <xacro:kuka_link
 			name="link1">

File: esercizio6/urdf/robot_kuka_generated.urdf (robot description, URDF)
Before this commit: robot robot_kuka, 8 links, 7 joints
Links:
- added link base_link; visual box size=10 0.6 0.02
- link link1: geometry visual cylinder length=0.2 radius=0.05
- link link2: geometry visual cylinder length=0.2 radius=0.05
- link link3: geometry visual cylinder length=0.2 radius=0.05
- link link4: geometry visual cylinder length=0.2 radius=0.05
- link link5: geometry visual cylinder length=0.2 radius=0.05
- link link6: geometry visual cylinder length=0.2 radius=0.05
- link link7: geometry visual cylinder length=0.2 radius=0.05
- link link_ee: geometry visual cylinder length=0.2 radius=0.05
Joints:
- added joint joint0: type prismatic, parent base_link, child link1, origin xyz=0 0 0, axis 1 0 0, limit lower=-5 upper=5 effort=176 velocity=0.1

File: esercizio6/urdf/robot_kuka_macro.xacro (robot description, xacro)
@@ -1,4 +1,17 @@
 <?xml version="1.0"?>
   <robot name="robot_kuka_macro" xmlns:xacro="http://wiki.ros.org/xacro">
+	<xacro:macro name="base_link_macro" params="base_link_name">
+		<link name="${base_link_name}">
+			<visual>
+				<geometry>
+					<box size="10 0.6 0.02"/>
+				</geometry>
+				<origin rpy="0 0 0" xyz="0 0 0"/>
+					<material name="yellow">
+						<color rgba="1 1 0 1"/>
+					</material>
+			</visual>
+		</link>
+	</xacro:macro>
 	<xacro:macro name="kuka_link" params="name *geometry *origin *orient  *material">
 		<link name="${name}">
@@ -9,8 +22,4 @@
 				<xacro:insert_block name="material" />
 		  </visual>
-		  <collision>
-				<xacro:insert_block name="geometry" />
-				<xacro:insert_block name="origin" />
-			</collision>
 	  </link>
 	</xacro:macro>
